Commit message: script to publish a traj with a few points

File: reflexxes_controllers_tests/model/sevenbot.urdf.xacro (robot description, xacro)
@@ -29,5 +29,5 @@
       <parent link="${parent}"/>
       <child link="${child}"/>
-      <dynamics damping="0.1" friction="0.0"/>
+      <dynamics damping="0.01" friction="0.0"/>
       <limit effort="100" velocity="100.0" lower="-1.57" upper="1.57" />
     </joint>
